Commit message: fix: LiDAR implement.

File: src/astar_robot_description/urdf/astar_robot.urdf (robot description, URDF)
Before this commit: robot astar_robot, 3 links, 2 joints
Links:
- added link lidar_link; visual cylinder length=0.04 radius=0.05
Joints:
- added joint lidar_joint: type fixed, parent base_link, child lidar_link, origin xyz=0.1 0 0.07
